File: pcb-holey/holey/holey-L.kicad_pcb (KiCad board)
At the start: 2 copper layers, 159.6 x 99.6 mm, 589 parts

Commit message: Updating holey boards.
Parts:
- REF** (x589): footprint holey:MountingHole_3.2mm_M3_JustHole -> MountingHole:MountingHole_3.2mm_M3_JustHole
