File: pcb-holey/holey/holey-M.kicad_pcb (KiCad board)
At the start: 2 copper layers, 79.6 x 99.6 mm, 285 parts

Commit message: Updating holey boards.
Parts:
- REF** (x285): footprint holey:MountingHole_3.2mm_M3_JustHole -> MountingHole:MountingHole_3.2mm_M3_JustHole
