File: pcb-holey/holey/holey-S.kicad_pcb (KiCad board)
At the start: 2 copper layers, 79.6 x 49.6 mm, 135 parts

Commit message: Updating holey boards.
Parts:
- REF** (x135): footprint holey:MountingHole_3.2mm_M3_JustHole -> MountingHole:MountingHole_3.2mm_M3_JustHole
