File: pcb-uart-combiner/uart-combiner/uart-combiner.kicad_pcb (KiCad board)
At the start: 2 copper layers, 52 x 82 mm, 23 parts, among them J1 Conn_01x04, J2 Conn_01x04, J3 Conn_01x04, J4 Conn_01x04, J5 Conn_01x03, J6 Conn_01x03

Commit message: Working on MPPT combiner.
Parts:
- removed D5, D7: FAULT, Diode_SMD:D_0603_1608Metric
- removed D6: BLINK, Diode_SMD:D_0603_1608Metric
- removed J2, J3, J4: Conn_01x04, Connector_JST:JST_PH_B4B-PH-K_1x04_P2.00mm_Vertical
- removed R5, R6, R7: 2.2k, Resistor_SMD:R_0603_1608Metric
- added D10: ~, Diode_SMD:D_0603_1608Metric, F.Cu at (115.5, 101.0)
- added D11: ~, Diode_SMD:D_0603_1608Metric, F.Cu at (115.5, 91.0)
- added D9: ~, Diode_SMD:D_0603_1608Metric, F.Cu at (115.5, 111.5)
- added J7: Conn_01x03, Connector_JST:JST_PH_B3B-PH-K_1x03_P2.00mm_Vertical, F.Cu at (110.0, 123.8)
- added J8: Conn_01x03, Connector_JST:JST_PH_B3B-PH-K_1x03_P2.00mm_Vertical, F.Cu at (110.0, 103.2)
- added J9: Conn_01x03, Connector_JST:JST_PH_B3B-PH-K_1x03_P2.00mm_Vertical, F.Cu at (110.0, 93.0)
- added R10: 2.2k, Resistor_SMD:R_0603_1608Metric, F.Cu at (122.9, 101.0)
- added R11: 2.2k, Resistor_SMD:R_0603_1608Metric, F.Cu at (122.9, 91.0)
- added R9: 2.2k, Resistor_SMD:R_0603_1608Metric, F.Cu at (122.9, 111.5)
- D3: value BLINK -> SERVER GOOD
- D4: value FAULT -> IP GOOD
- D8: value BLINK -> ~
- J1: value Conn_01x04 -> Conn_01x03; footprint Connector_JST:JST_PH_B4B-PH-K_1x04_P2.00mm_Vertical -> Connector_JST:JST_PH_B3B-PH-K_1x03_P2.00mm_Vertical
- J5: value Conn_01x03 -> DBG UART
- J6: value Conn_01x03 -> SWD
- moved D8 38.0 mm to (115.5, 121.8), turned to 90 degrees
- moved R8 31.9 mm to (122.9, 121.8), turned to 90 degrees
- moved J1 19.8 mm to (110.0, 113.5)
- moved R4 18.2 mm to (150.0, 104.0), turned to 180 degrees
- moved R3 9.73 mm to (150.0, 110.2)
- moved D3 6.30 mm to (153.2, 110.2), turned to 180 degrees
- moved D4 2.54 mm to (153.2, 104.0), turned to 180 degrees
- moved J5 1.68 mm to (153.7, 84.2)
- moved J6 1.25 mm to (153.7, 95.0)
Connections:
- A1 pad 13: Net-(A1-GND-Pad13) -> GND
- A1 pad 18: Net-(A1-GND-Pad13) -> GND
- A1 pad 21: (no net) -> unconnected-(A1-NC-Pad21)
- A1 pad 22: (no net) -> unconnected-(A1-NC-Pad22)
- A1 pad 23: Net-(A1-GND-Pad13) -> GND
- A1 pad 24: (no net) -> unconnected-(A1-NC-Pad24)
- A1 pad 25: (no net) -> unconnected-(A1-NC-Pad25)
- A1 pad 26: (no net) -> unconnected-(A1-NC-Pad26)_1
- A1 pad 27: (no net) -> unconnected-(A1-NC-Pad27)_1
- A1 pad 28: Net-(A1-GND-Pad13) -> GND
- A1 pad 29: (no net) -> unconnected-(A1-NC-Pad29)_1
- A1 pad 3: Net-(A1-GND-Pad13) -> GND
- A1 pad 38: Net-(A1-GND-Pad13) -> GND
- A1 pad 8: Net-(A1-GND-Pad13) -> GND
- A1 pad D2: Net-(A1-GND-Pad13) -> GND
- J1 pad 2: Net-(A1-GPIO15) -> Net-(A1-GPIO11)
- J1 pad 3: Net-(A1-GPIO14) -> Net-(A1-GPIO10)
- J5 pad MP: (no net) -> GND
- J6 pad MP: (no net) -> GND
- R8 pad 1: Net-(A1-GPIO7) -> Net-(A1-GPIO15)
Routing:
- net Net-(A1-GPIO3): track 0.00 -> 40.4 mm
- net Net-(A1-GPIO2): track 0.00 -> 36.7 mm
- net Net-(A1-GPIO0): track 0.00 -> 30.1 mm
- net Net-(A1-GPIO1): track 0.00 -> 29.9 mm
- net Net-(A1-SWCLK): track 0.00 -> 29.3 mm
- net Net-(A1-GPIO13): track 0.00 -> 18.7 mm
- net Net-(A1-GPIO5): track 0.00 -> 18.0 mm
- net Net-(A1-GPIO11): track 0.00 -> 17.9 mm
- net Net-(A1-GPIO14): track 0.00 -> 17.9 mm
- net Net-(A1-GPIO4): track 0.00 -> 17.8 mm
- net Net-(A1-GPIO7): track 0.00 -> 17.7 mm
- net Net-(A1-GPIO10): track 0.00 -> 17.7 mm
- net Net-(A1-GPIO8): track 0.00 -> 17.5 mm
- net Net-(A1-SWDIO): track 0.00 -> 15.4 mm
- net Net-(A1-GPIO6): track 0.00 -> 8.97 mm
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- added copper zone on F.Cu, net GND

Commit message: V1 mostly done.
Parts:
- added D5: RUNNING, Diode_SMD:D_0603_1608Metric, F.Cu at (153.3, 115.8)
- added R5: 2.2k, Resistor_SMD:R_0603_1608Metric, F.Cu at (150.0, 115.8)
- added TP1: GND, TestPoint:TestPoint_Keystone_5019_Miniature, F.Cu at (118.6, 75.0)
- moved D3 0.05 mm to (153.3, 110.2)
- moved D4 0.05 mm to (153.3, 104.0)
Connections:
- A1 pad 34: unconnected-(A1-GPIO28_ADC2-Pad34) -> Net-(A1-GPIO28_ADC2)
Routing:
- net Net-(A1-GPIO28_ADC2): track 0.00 -> 27.2 mm, vias 0 -> 1
- net Net-(D5-A): track 0.00 -> 1.69 mm
- net GND: vias 0 -> 1
- added copper zone on B.Cu, net GND
Other:
- board size 52 x 82 mm -> 52.2 x 82.2 mm
- board text added: "MPPT Relay v1.0 (c) devbotas"
